File: MRCS-Dual-3-Position-Semaphore-Controller v13.sch (EAGLE design)
At the start: 26 parts, among them J1 5 VDC, J2 Input, M1 SMALL_SERVO, M2 SMALL_SERVO

Commit message: updates based on Holbrook's crew
added 3.5mm power terminal, added filter caps for noisy servos
Parts:
- added CON1: (no value), SPCoast:CONNECTOR-M023.5MM-LOCK
Connections:
- net 5V: now also CON1.B
- net GND: now also CON1.A
Other:
- note added: "+5 GND"
Changed lines of the file:
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@@
 <part name="C3" library="SPCoast" deviceset="CAP*" device="PTH1" value=".01 uF"/>
 <part name="C4" library="SPCoast" deviceset="CAP-POL*" device="PTH-5MM" value="220 uF @ 35"/>
+<part name="CON1" library="SPCoast" deviceset="CONNECTOR-M02" device="3.5MM-LOCK"/>
+<part name="GND5" library="SparkFun-Aesthetics" deviceset="GND" device=""/>
 </parts>
 <sheets>
@@
 <text x="157.48" y="17.78" size="3.81" layer="94" font="vector">Seth Neumann, Earl Girbovan</text>
 <text x="236.22" y="-2.54" size="2.54" layer="91">1.3</text>
+<text x="1.27" y="29.21" size="1.778" layer="91">+5
+GND</text>
 </plain>
 <instances>
@@
 <instance part="C3" gate="C1" x="132.08" y="132.08"/>
 <instance part="C4" gate="C1" x="45.72" y="5.08"/>
+<instance part="CON1" gate="J" x="12.7" y="30.48"/>
+<instance part="GND5" gate="1" x="20.32" y="22.86"/>
 </instances>
 <busses>
@@
 <pinref part="C2" gate="C1" pin="2"/>
 <wire x1="134.62" y1="152.4" x2="134.62" y2="154.94" width="0.1524" layer="91"/>
+</segment>
+<segment>
+<pinref part="CON1" gate="J" pin="A"/>
+<wire x1="17.78" y1="30.48" x2="20.32" y2="30.48" width="0.4064" layer="91"/>
+<pinref part="GND5" gate="1" pin="GND"/>
+<wire x1="20.32" y1="30.48" x2="20.32" y2="25.4" width="0.4064" layer="91"/>
 </segment>
 </net>
@@
 <wire x1="45.72" y1="7.62" x2="45.72" y2="12.7" width="0.4064" layer="91"/>
 <junction x="45.72" y="12.7"/>
-</segment>
-<segment>
+<pinref part="CON1" gate="J" pin="B"/>
+<wire x1="17.78" y1="33.02" x2="45.72" y2="33.02" width="0.4064" layer="91"/>
+<wire x1="45.72" y1="33.02" x2="45.72" y2="12.7" width="0.4064" layer="91"/>
+</segment>
+<segment>
